File: rados (copy).kicad_pcb (KiCad board)
At the start: 2 copper layers, 156 parts, among them J1 HEADER, J10 STEPSTICK, J11 STEPSTICK, J12 STEPSTICK, J13 MICROSD_SLOT_TFP09-2-12B, J2 HEADER, J3 HEADER, J4 STEPSTICK, J5 STEPSTICK, J6 STEPSTICK, J7 HEADER, J8 HEADER, J9 HEADER, P1 CONN_01X02, P10 CONN_01X04, P11 CONN_01X04, P12 CONN_01X04, P13 EXT_SD, P14 LCD, P15 LIMIT_SWITCHES, P16 LIMIT_SWITCHES_V, P17 CONN_01X03, P18 CONN_01X03, P19 CONN_01X03, P2 CONN_01X02, P20 CONN_01X03, P21 THERMISTORS, P22 CONN_01X05, P3 CONN_01X02, P4 CONN_01X02, P5 HP_MOSFETS, P6 MP_MOSFETS, P7 CONN_02X04, P8 CONN_01X04, P9 CONN_01X04, Q1 2N7002P, Q10 2N7002P, Q11 2N7002P, Q12 BC846BPDW1, Q13 BC846BPDW1, Q14 SI2318CDS-T1-GE3, Q15 IRFB7545PbF, Q16 2N7002P, Q17 2N7002P, Q18 BC846BPDW1, Q19 BC846BPDW1, Q2 2N7002P, Q20 SI2318CDS-T1-GE3, Q21 IRFB7545PbF, Q3 2N7002P, Q4 BC846BPDW1, Q5 BC846BPDW1, Q6 BC846BPDW1, Q7 IRFB7545PbF, Q8 SI2318CDS-T1-GE3, Q9 IRFB7545PbF, SW1 RESET, U1 MC34063, U2 24LC256

Commit message: More routing
Parts:
- C12, C13, C14, C15, C16, C17: footprint geda-footprints:ELCO-8mm -> armin-footprints:ELCO-8mm
- D11, D15, D7: footprint geda-footprints:LL-34 -> armin-footprints:LL-34
- D12, D16, D2, D6, D8: footprint geda-footprints:DO214AC -> armin-footprints:DO214AC
- Q1, Q10, Q11, Q14, Q16, Q17, Q2, Q20, Q3, Q8: footprint geda-footprints:SOT23_3L -> armin-footprints:SOT23_3L
- Q12, Q13, Q18, Q19, Q4, Q5, Q6: footprint geda-footprints:SC70_6L -> armin-footprints:SC70_6L
- Q15, Q21, Q7, Q9: footprint geda-footprints:TO-220 -> armin-footprints:TO-220
- moved D10 179.5 mm to (96.0, 75.2), turned to 90 degrees
- moved D14 177.1 mm to (96.0, 64.2), turned to 90 degrees
- moved Q17 176.6 mm to (99.0, 65.0), turned to 180 degrees
- moved R23 176.6 mm to (96.2, 71.8), turned to 90 degrees
- moved Q19 174.5 mm to (99.2, 61.4), turned to 180 degrees
- moved R31 173.3 mm to (96.3, 60.9), turned to 90 degrees
- moved Q11 171.3 mm to (98.7, 76.3), turned to 180 degrees
- moved R29 171.0 mm to (96.2, 67.5), turned to 90 degrees
- moved R5 163.5 mm to (98.9, 55.5)
- moved C6 154.3 mm to (101.3, 73.4), turned to 90 degrees
- moved R17 149.7 mm to (106.7, 81.3)
- moved Q13 147.7 mm to (98.8, 73.2), turned to 180 degrees
- moved R19 142.3 mm to (98.8, 71.0)
- moved R21 140.3 mm to (96.2, 78.5), turned to 90 degrees
- moved R25 124.5 mm to (106.7, 66.0)
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Connections:
- net LCD-4 renamed Net-(SHIELD1-Pad44)
- net LCD-5 renamed Net-(SHIELD1-Pad45)
- net LCD-6 renamed Net-(SHIELD1-Pad46)
- net LCD-7 renamed Net-(SHIELD1-Pad47)
- J1 pad 2: Net-(J1-Pad2) -> +3V3
- J1 pad 4: Net-(J1-Pad4) -> +3V3
- J1 pad 6: Net-(J1-Pad6) -> +3V3
- J2 pad 2: Net-(J2-Pad2) -> +3V3
- J2 pad 4: Net-(J2-Pad4) -> +3V3
- J2 pad 6: Net-(J2-Pad6) -> +3V3
- J3 pad 2: Net-(J3-Pad2) -> +3V3
- J3 pad 4: Net-(J3-Pad4) -> +3V3
- J3 pad 6: Net-(J3-Pad6) -> +3V3
- J4 pad 2: Net-(J1-Pad2) -> Net-(J1-Pad1)
- J4 pad 3: Net-(J1-Pad4) -> Net-(J1-Pad3)
- J4 pad 4: Net-(J1-Pad6) -> Net-(J1-Pad5)
- J5 pad 2: Net-(J2-Pad2) -> Net-(J2-Pad1)
- J5 pad 3: Net-(J2-Pad4) -> Net-(J2-Pad3)
- J5 pad 4: Net-(J2-Pad6) -> Net-(J2-Pad5)
- J6 pad 2: Net-(J3-Pad2) -> Net-(J3-Pad1)
- J6 pad 3: Net-(J3-Pad4) -> Net-(J3-Pad3)
- J6 pad 4: Net-(J3-Pad6) -> Net-(J3-Pad5)
- J7 pad 1: Net-(J7-Pad1) -> Net-(J10-Pad2)
- J7 pad 2: Net-(J10-Pad2) -> +3V3
- J7 pad 3: Net-(J7-Pad3) -> Net-(J10-Pad3)
- J7 pad 4: Net-(J10-Pad3) -> +3V3
- J7 pad 5: Net-(J7-Pad5) -> Net-(J10-Pad4)
- J7 pad 6: Net-(J10-Pad4) -> +3V3
- J8 pad 1: Net-(J8-Pad1) -> Net-(J11-Pad2)
- J8 pad 2: Net-(J11-Pad2) -> +3V3
- J8 pad 3: Net-(J8-Pad3) -> Net-(J11-Pad3)
- J8 pad 4: Net-(J11-Pad3) -> +3V3
- J8 pad 5: Net-(J8-Pad5) -> Net-(J11-Pad4)
- J8 pad 6: Net-(J11-Pad4) -> +3V3
- J9 pad 1: Net-(J9-Pad1) -> Net-(J12-Pad2)
- J9 pad 2: Net-(J12-Pad2) -> +3V3
- J9 pad 3: Net-(J9-Pad3) -> Net-(J12-Pad3)
- J9 pad 4: Net-(J12-Pad3) -> +3V3
- J9 pad 5: Net-(J9-Pad5) -> Net-(J12-Pad4)
- J9 pad 6: Net-(J12-Pad4) -> +3V3
- P17 pad 1: GND -> +3V3
- P17 pad 2: +3V3 -> GND
- P18 pad 1: GND -> +3V3
- P18 pad 2: +3V3 -> GND
- P19 pad 1: GND -> +3V3
- P19 pad 2: +3V3 -> GND
- P20 pad 1: GND -> +3V3
- P20 pad 2: +3V3 -> GND
- SHIELD1 pad 0: Y-STEP -> HP-FET3
- SHIELD1 pad 1: Net-(SHIELD1-Pad1) -> Y-STEP
- SHIELD1 pad 15: Net-(SHIELD1-Pad15) -> MP-FET1
- SHIELD1 pad 16: Y-DIR -> LP-FET1
- SHIELD1 pad 17: MP-FET1 -> LP-FET2
- SHIELD1 pad 18: LP-FET2 -> X-STEP
- SHIELD1 pad 19: LP-FET1 -> X-DIR
- SHIELD1 pad 2: Net-(SHIELD1-Pad2) -> Y-DIR
- SHIELD1 pad 22: Y-EN -> X-
- SHIELD1 pad 23: X-DIR -> X+
- SHIELD1 pad 24: X-STEP -> Y-
- SHIELD1 pad 25: Net-(SHIELD1-Pad25) -> Y+
- SHIELD1 pad 26: X-EN -> Z-
- SHIELD1 pad 27: Net-(SHIELD1-Pad27) -> Z+
- SHIELD1 pad 28: X- -> PROBE
- SHIELD1 pad 3: Net-(SHIELD1-Pad3) -> Y-EN
- SHIELD1 pad 30: Y- -> Net-(SHIELD1-Pad30)
- SHIELD1 pad 32: Z- -> Net-(SHIELD1-Pad32)
- SHIELD1 pad 33: Net-(SHIELD1-Pad33) -> LCD-D4
- SHIELD1 pad 34: X+ -> LCD-D5
- SHIELD1 pad 35: Net-(SHIELD1-Pad35) -> LCD-D6
- SHIELD1 pad 36: Y+ -> LCD-D7
- SHIELD1 pad 37: Net-(SHIELD1-Pad37) -> LCD-E
- SHIELD1 pad 38: Z+ -> LCD-RS
- SHIELD1 pad 40: Net-(SHIELD1-Pad40) -> X-EN
- SHIELD1 pad 42: LCD-RS -> Net-(SHIELD1-Pad42)
- SHIELD1 pad 43: LCD-E -> Net-(SHIELD1-Pad43)
- SHIELD1 pad 49: E3-EN -> Net-(SHIELD1-Pad49)
- SHIELD1 pad 51: E3-STEP -> Net-(SHIELD1-Pad51)
- SHIELD1 pad 53: E3-DIR -> Net-(SHIELD1-Pad53)
- SHIELD1 pad 7: HP-FET3 -> Net-(SHIELD1-Pad7)
- SHIELD1 pad AD10: E2-STEP -> AUX-4
- SHIELD1 pad AD11: T4 -> T0
- SHIELD1 pad AD12: T3 -> T1
- SHIELD1 pad AD14: T1 -> T3
- SHIELD1 pad AD15: T0 -> T4
- SHIELD1 pad AD5: E2-EN -> Net-(SHIELD1-PadAD5)
- SHIELD1 pad AD6: E1-DIR -> Net-(SHIELD1-PadAD6)
- SHIELD1 pad AD7: E1-STEP -> AUX-1
- SHIELD1 pad AD8: E1-EN -> AUX-2
- SHIELD1 pad AD9: E2-DIR -> AUX-3
Routing:
- net +3V3: track 0.00 -> 85.0 mm
- net Vsupply: track 261.0 -> 319.8 mm, vias 0 -> 1
- net AUX-1: track 0.00 -> 42.0 mm
- net AUX-2: track 0.00 -> 35.0 mm
- net AUX-3: track 0.00 -> 32.6 mm
- net AUX-4: track 0.00 -> 28.6 mm
- net T0: track 0.00 -> 27.1 mm
- net Z-EN: track 0.00 -> 24.5 mm
- net T2: track 0.00 -> 22.1 mm
- net T1: track 0.00 -> 21.4 mm
- net T3: track 0.00 -> 13.4 mm
- net MP-OUT1: track 0.00 -> 12.7 mm
- net T4: track 0.00 -> 10.0 mm
- net Z-STEP: track 0.00 -> 7.95 mm
- net GND: track 23.5 -> 31.5 mm, vias 2 -> 6
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Other:
- board outline added: 83 x 106 mm
- net class Default: clearance 0.15 -> 0.1524; trace_width 0.15 -> 0.1524
- rule trace_clearance: 0.15 -> 0.1524
- rule trace_min: 0.15 -> 0.1524

Commit message: Routing almost finished
Parts:
- removed R32, R33, R34: 10K, Resistors_SMD:R_0603
- added C33: 10uF, Capacitors_SMD:C_0805, F.Cu at (92.4, 25.4)
- D10, D13, D14, D17, D3, D4, D5, D9: footprint geda-footprints:0603diode -> armin-footprints:0603diode
- L1: value 100uF -> 100uH
- R10: value 1K8 -> 4K7; footprint Resistors_SMD:R_0603 -> Resistors_SMD:R_0805
- U1, U2: footprint geda-footprints:SOIC8 -> armin-footprints:SOIC8
- moved Q4 173.2 mm to (98.8, 95.3), turned to 180 degrees
- moved C5 169.7 mm to (95.9, 56.5), turned to 90 degrees
- moved D3 167.1 mm to (96.0, 97.5), turned to 90 degrees
- moved R27 166.5 mm to (98.9, 59.2)
- moved Q1 165.3 mm to (99.0, 98.2), turned to 180 degrees
- moved C11 161.4 mm to (101.2, 61.2), turned to 90 degrees
- moved R7 153.4 mm to (98.7, 93.2)
- moved R10 152.3 mm to (96.2, 100.5), turned to 90 degrees
- moved R13 147.6 mm to (96.2, 94.0), turned to 90 degrees
- moved R4 145.3 mm to (102.1, 99.8), turned to 90 degrees
- moved C9 137.9 mm to (101.3, 95.1), turned to 90 degrees
- moved R42 100.3 mm to (92.8, 27.4), turned to 180 degrees
- moved D17 94.6 mm to (89.0, 27.6), turned to 180 degrees
- moved C32 48.8 mm to (107.0, 106.3), turned to 180 degrees
- moved D2 47.0 mm to (105.6, 113.8)
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Connections:
- C31 pad 2: Net-(C31-Pad2) -> GND
- J11 pad 1: E1-EN -> E2-EN
- J11 pad 7: E1-STEP -> E2-STEP
- J11 pad 8: E1-DIR -> E2-DIR
- J12 pad 1: E2-EN -> E1-EN
- J12 pad 7: E2-STEP -> E1-STEP
- J12 pad 8: E2-DIR -> E1-DIR
- R35 pad 1: Net-(R35-Pad1) -> +3V3
- R36 pad 1: Net-(R35-Pad1) -> +3V3
- SHIELD1 pad 1: Y-STEP -> Y-EN
- SHIELD1 pad 29: Net-(SHIELD1-Pad29) -> STATUS-LED
- SHIELD1 pad 3: Y-EN -> Y-STEP
- SHIELD1 pad 34: LCD-D5 -> LCD-D7
- SHIELD1 pad 36: LCD-D7 -> LCD-E
- SHIELD1 pad 37: LCD-E -> LCD-D5
- SHIELD1 pad 39: Net-(SHIELD1-Pad39) -> ENC-B
- SHIELD1 pad 41: STATUS-LED -> ENC-A
- SHIELD1 pad 44: Net-(SHIELD1-Pad44) -> E3-EN
- SHIELD1 pad 45: Net-(SHIELD1-Pad45) -> E3-STEP
- SHIELD1 pad 46: Net-(SHIELD1-Pad46) -> E3-DIR
- SHIELD1 pad 48: ENC-SW -> Net-(SHIELD1-Pad48)
- SHIELD1 pad 50: ENC-B -> Net-(SHIELD1-Pad50)
- SHIELD1 pad 52: ENC-A -> Net-(SHIELD1-Pad52)
- SHIELD1 pad 7: Net-(SHIELD1-Pad7) -> HP-FET1
- SHIELD1 pad 8: HP-FET1 -> Z-STEP
- SHIELD1 pad 9: Z-STEP -> ENC-SW
- SHIELD1 pad AD0: Net-(SHIELD1-PadAD0) -> E1-DIR
- SHIELD1 pad AD1: Net-(SHIELD1-PadAD1) -> E1-STEP
- SHIELD1 pad AD2: Net-(SHIELD1-PadAD2) -> E1-EN
- SHIELD1 pad AD3: Net-(SHIELD1-PadAD3) -> E2-DIR
- SHIELD1 pad AD4: Net-(SHIELD1-PadAD4) -> E2-STEP
- SHIELD1 pad AD5: Net-(SHIELD1-PadAD5) -> E2-EN
- SW1 pad 2: Net-(C31-Pad2) -> GND
Routing:
- net +3V3: track 85.0 -> 533.1 mm, vias 0 -> 3
- net +12V: track 31.5 -> 230.0 mm
- net SD2-CS: track 0.00 -> 80.8 mm
- net SD-CS: track 0.00 -> 77.6 mm
- net Net-(D2-Pad1): track 0.00 -> 71.4 mm
- net E1-DIR: track 0.00 -> 61.3 mm
- net E1-STEP: track 0.00 -> 61.1 mm
- net RESET: track 0.00 -> 48.9 mm
- net ENC-SW: track 0.00 -> 48.9 mm
- net E1-EN: track 0.00 -> 48.5 mm
- net GND: track 31.5 -> 75.7 mm, vias 6 -> 32
- net E3-EN: track 0.00 -> 43.5 mm
- net +5V: track 0.00 -> 39.0 mm
- net E2-EN: track 0.00 -> 37.3 mm
- net SD-SCK: track 48.5 -> 83.9 mm
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Other:
- board size 83 x 106 mm -> 83.2 x 106 mm
