File: power.sch (KiCad schematic (older format))
At the start: 19 parts, among them P1 CONN_01X02, P2 CONN_01X02, P3 CONN_01X02, P4 CONN_01X02, U1 MC34063

Commit message: More schematics, some layout
Connections:
- net at R1.2, U1.1 (SWC), U1.7 (Isense): now also U1.8 (DRC)
Changed lines of the file:
@@
 	1    0    0    -1
 $EndComp
+Connection ~ 2025 1725
 $EndSCHEMATC

Commit message: more placement and routing
Parts:
- P3, P4: footprint geda-footprints:CON_SCRW_2_PIN -> geda-footprints:CON_HDR_1x2
Changed lines of the file:
@@
 EESchema Schematic File Version 2
+LIBS:led_reverse
 LIBS:arduino_shieldsNCL
 LIBS:otheruse_transistors
@@
 $EndComp
 $Comp
-L +12V #PWR04
+L +12V #PWR06
 U 1 1 568AC408
 P 5150 1925
-F 0 "#PWR04" H 5150 1775 50  0001 C CNN
+F 0 "#PWR06" H 5150 1775 50  0001 C CNN
 F 1 "+12V" H 5168 2099 50  0000 C CNN
 F 2 "" H 5150 1925 50  0000 C CNN
@@
 $EndComp
 $Comp
-L GND #PWR05
+L GND #PWR07
 U 1 1 568AE875
 P 1425 4450
-F 0 "#PWR05" H 1425 4200 50  0001 C CNN
+F 0 "#PWR07" H 1425 4200 50  0001 C CNN
 F 1 "GND" H 1433 4276 50  0000 C CNN
 F 2 "" H 1425 4450 50  0000 C CNN
@@
 $EndComp
 $Comp
-L GND #PWR06
+L GND #PWR08
 U 1 1 568AE8A5
 P 2800 2325
-F 0 "#PWR06" H 2800 2075 50  0001 C CNN
+F 0 "#PWR08" H 2800 2075 50  0001 C CNN
 F 1 "GND" H 2808 2151 50  0000 C CNN
 F 2 "" H 2800 2325 50  0000 C CNN
@@
 	1500 4350 1425 4350
 $Comp
-L Vsupply #P07
+L Vsupply #P09
 U 1 1 568AD53F
 P 4750 1225
-F 0 "#P07" H 4750 1225 60  0001 C CNN
+F 0 "#P09" H 4750 1225 60  0001 C CNN
 F 1 "Vsupply" H 4750 1175 34  0000 C CNN
 F 2 "" H 4750 1225 60  0000 C CNN
@@
 $EndComp
 $Comp
-L Vsupply #P08
+L Vsupply #P010
 U 1 1 568AD70E
 P 1525 1775
-F 0 "#P08" H 1525 1775 60  0001 C CNN
+F 0 "#P010" H 1525 1775 60  0001 C CNN
 F 1 "Vsupply" H 1525 1725 34  0000 C CNN
 F 2 "" H 1525 1775 60  0000 C CNN
@@
 $EndComp
 $Comp
-L GND #PWR09
+L GND #PWR011
 U 1 1 568ADBA9
 P 1450 3800
-F 0 "#PWR09" H 1450 3550 50  0001 C CNN
+F 0 "#PWR011" H 1450 3550 50  0001 C CNN
 F 1 "GND" H 1458 3626 50  0000 C CNN
 F 2 "" H 1450 3800 50  0000 C CNN
@@
 	1525 3700 1450 3700
 $Comp
-L Vsupply #P010
+L Vsupply #P012
 U 1 1 568ADC9C
 P 2125 3550
-F 0 "#P010" H 2125 3550 60  0001 C CNN
+F 0 "#P012" H 2125 3550 60  0001 C CNN
 F 1 "Vsupply" H 2125 3500 34  0000 C CNN
 F 2 "" H 2125 3550 60  0000 C CNN
@@
 $EndComp
 $Comp
-L Vheatbed #P011
+L Vheatbed #P013
 U 1 1 568AE31D
 P 2100 4200
-F 0 "#P011" H 2100 4200 60  0001 C CNN
+F 0 "#P013" H 2100 4200 60  0001 C CNN
 F 1 "Vheatbed" H 2100 4150 34  0000 C CNN
 F 2 "" H 2100 4200 60  0000 C CNN
@@
 F 0 "P3" H 1275 5175 50  0000 C CNN
 F 1 "CONN_01X02" H 1194 5160 50  0001 C CNN
-F 2 "geda-footprints:CON_SCRW_2_PIN" H 1275 5350 50  0001 C CNN
+F 2 "geda-footprints:CON_HDR_1x2" H 1275 5350 50  0001 C CNN
 F 3 "" H 1275 5350 50  0000 C CNN
 	1    1275 5350
@@
 $EndComp
 $Comp
-L GND #PWR012
+L GND #PWR014
 U 1 1 568AE68D
 P 1475 5400
-F 0 "#PWR012" H 1475 5150 50  0001 C CNN
+F 0 "#PWR014" H 1475 5150 50  0001 C CNN
 F 1 "GND" H 1483 5226 50  0000 C CNN
 F 2 "" H 1475 5400 50  0000 C CNN
@@
 	1475 5300 1650 5300
 $Comp
-L Vsupply #P013
+L Vsupply #P015
 U 1 1 568AE69B
 P 1650 5150
-F 0 "#P013" H 1650 5150 60  0001 C CNN
+F 0 "#P015" H 1650 5150 60  0001 C CNN
 F 1 "Vsupply" H 1650 5100 34  0000 C CNN
 F 2 "" H 1650 5150 60  0000 C CNN
@@
 F 0 "P4" H 1275 6250 50  0000 C CNN
 F 1 "CONN_01X02" H 1194 6235 50  0001 C CNN
-F 2 "geda-footprints:CON_SCRW_2_PIN" H 1275 6425 50  0001 C CNN
+F 2 "geda-footprints:CON_HDR_1x2" H 1275 6425 50  0001 C CNN
 F 3 "" H 1275 6425 50  0000 C CNN
 	1    1275 6425
@@
 $EndComp
 $Comp
-L GND #PWR014
+L GND #PWR016
 U 1 1 568AE860
 P 1475 6475
-F 0 "#PWR014" H 1475 6225 50  0001 C CNN
+F 0 "#PWR016" H 1475 6225 50  0001 C CNN
 F 1 "GND" H 1483 6301 50  0000 C CNN
 F 2 "" H 1475 6475 50  0000 C CNN
@@
 	1475 6375 1650 6375
 $Comp
-L +12V #PWR015
+L +12V #PWR017
 U 1 1 568BD457
 P 1650 6375
-F 0 "#PWR015" H 1650 6225 50  0001 C CNN
+F 0 "#PWR017" H 1650 6225 50  0001 C CNN
 F 1 "+12V" H 1668 6549 50  0000 C CNN
 F 2 "" H 1650 6375 50  0000 C CNN

Commit message: More routing
Parts:
- D2: footprint geda-footprints:DO214AC -> armin-footprints:DO214AC
- L1: value 100uF -> 100uH
- U1: footprint geda-footprints:SOIC8 -> armin-footprints:SOIC8
Changed lines of the file:
@@
 F 0 "U1" H 2425 2475 34  0000 C BNN
 F 1 "MC34063" H 2425 2150 34  0000 C BNN
-F 2 "geda-footprints:SOIC8" H 2025 2100 60  0001 C CNN
+F 2 "armin-footprints:SOIC8" H 2025 2100 60  0001 C CNN
 F 3 "" H 2025 2100 60  0000 C CNN
 	1    2025 2100
@@
 P 3575 1825
 F 0 "L1" V 3650 1800 50  0000 L CNN
-F 1 "100uF" V 3525 1725 50  0000 L CNN
+F 1 "100uH" V 3525 1725 50  0000 L CNN
 F 2 "geda-footprints:INDUCTOR_AIUR06" H 3575 1825 50  0001 C CNN
 F 3 "" H 3575 1825 50  0000 C CNN
@@
 F 0 "D2" H 4862 2907 34  0000 C CNN
 F 1 "ES1G" H 4862 2838 34  0000 C CNN
-F 2 "geda-footprints:DO214AC" H 4750 2675 60  0001 C CNN
+F 2 "armin-footprints:DO214AC" H 4750 2675 60  0001 C CNN
 F 3 "" H 4750 2675 60  0000 C CNN
 	1    4750 2675

Commit message: Added 3d models
Parts:
- D1: footprint geda-footprints:SMB -> armin-footprints:DO214AA
- F1, F2: footprint geda-footprints:FUSEHOLDER_MINI_KEYSTONE_3557 -> armin-footprints:FUSEHOLDER_MINI_KEYSTONE_3557
- JP1: footprint geda-footprints:CON_HDR_1x3 -> armin-footprints:CON_HDR_1x3_2.54mm
- JP2, P3, P4: footprint geda-footprints:CON_HDR_1x2 -> armin-footprints:CON_HDR_1x2_2.54mm
- L1: footprint geda-footprints:INDUCTOR_AIUR06 -> armin-footprints:INDUCTOR_AIUR06
- P1, P2: footprint geda-footprints:CON_WURTH_WR_TBL_313_2 -> armin-footprints:CON_PHOENIX_MSTBA-2.5-2-G-5.08
Changed lines of the file:
@@
 F 0 "D1" H 3450 2100 34  0000 L BNN
 F 1 "STPS3L40UF" H 3375 2300 34  0000 L BNN
-F 2 "geda-footprints:SMB" H 3425 2175 60  0001 C CNN
+F 2 "armin-footprints:DO214AA" H 3425 2175 60  0001 C CNN
 F 3 "" H 3425 2175 60  0000 C CNN
 	1    3425 2175
@@
 F 0 "L1" V 3650 1800 50  0000 L CNN
 F 1 "100uH" V 3525 1725 50  0000 L CNN
-F 2 "geda-footprints:INDUCTOR_AIUR06" H 3575 1825 50  0001 C CNN
+F 2 "armin-footprints:INDUCTOR_AIUR06" H 3575 1825 50  0001 C CNN
 F 3 "" H 3575 1825 50  0000 C CNN
 	1    3575 1825
@@
 F 0 "JP1" H 4400 2065 50  0000 C CNN
 F 1 "VSEL" H 4400 1973 50  0000 C CNN
-F 2 "geda-footprints:CON_HDR_1x3" H 4400 1825 50  0001 C CNN
+F 2 "armin-footprints:CON_HDR_1x3_2.54mm" H 4400 1825 50  0001 C CNN
 F 3 "" H 4400 1825 50  0000 C CNN
 	1    4400 1825
@@
 F 0 "JP2" H 5850 2890 50  0000 C CNN
 F 1 "BOARD_POWER" H 5850 2798 50  0000 C CNN
-F 2 "geda-footprints:CON_HDR_1x2" H 5850 2625 50  0001 C CNN
+F 2 "armin-footprints:CON_HDR_1x2_2.54mm" H 5850 2625 50  0001 C CNN
 F 3 "" H 5850 2625 50  0000 C CNN
 	1    5850 2625
@@
 F 0 "P1" H 1250 4225 50  0000 C CNN
 F 1 "CONN_01X02" H 1144 4210 50  0001 C CNN
-F 2 "geda-footprints:CON_WURTH_WR_TBL_313_2" H 1225 4400 50  0001 C CNN
+F 2 "armin-footprints:CON_PHOENIX_MSTBA-2.5-2-G-5.08" H 1225 4400 50  0001 C CNN
 F 3 "" H 1225 4400 50  0000 C CNN
 	1    1225 4400
@@
 F 0 "F1" H 1750 4591 50  0000 C CNN
 F 1 "FUSE" H 1750 4499 50  0000 C CNN
-F 2 "geda-footprints:FUSEHOLDER_MINI_KEYSTONE_3557" H 1750 4350 50  0001 C CNN
+F 2 "armin-footprints:FUSEHOLDER_MINI_KEYSTONE_3557" H 1750 4350 50  0001 C CNN
 F 3 "" H 1750 4350 50  0000 C CNN
 	1    1750 4350
@@
 F 0 "P2" H 1250 3575 50  0000 C CNN
 F 1 "CONN_01X02" H 1169 3560 50  0001 C CNN
-F 2 "geda-footprints:CON_WURTH_WR_TBL_313_2" H 1250 3750 50  0001 C CNN
+F 2 "armin-footprints:CON_PHOENIX_MSTBA-2.5-2-G-5.08" H 1250 3750 50  0001 C CNN
 F 3 "" H 1250 3750 50  0000 C CNN
 	1    1250 3750
@@
 F 0 "F2" H 1775 3941 50  0000 C CNN
 F 1 "FUSE" H 1775 3849 50  0000 C CNN
-F 2 "geda-footprints:FUSEHOLDER_MINI_KEYSTONE_3557" H 1775 3700 50  0001 C CNN
+F 2 "armin-footprints:FUSEHOLDER_MINI_KEYSTONE_3557" H 1775 3700 50  0001 C CNN
 F 3 "" H 1775 3700 50  0000 C CNN
 	1    1775 3700
@@
 F 0 "P3" H 1275 5175 50  0000 C CNN
 F 1 "CONN_01X02" H 1194 5160 50  0001 C CNN
-F 2 "geda-footprints:CON_HDR_1x2" H 1275 5350 50  0001 C CNN
+F 2 "armin-footprints:CON_HDR_1x2_2.54mm" H 1275 5350 50  0001 C CNN
 F 3 "" H 1275 5350 50  0000 C CNN
 	1    1275 5350
@@
 F 0 "P4" H 1275 6250 50  0000 C CNN
 F 1 "CONN_01X02" H 1194 6235 50  0001 C CNN
-F 2 "geda-footprints:CON_HDR_1x2" H 1275 6425 50  0001 C CNN
+F 2 "armin-footprints:CON_HDR_1x2_2.54mm" H 1275 6425 50  0001 C CNN
 F 3 "" H 1275 6425 50  0000 C CNN
 	1    1275 6425

Commit message: More 3d stuff
Parts:
- C4: footprint Resistors_SMD:R_1210 -> Capacitors_SMD:C_1210
Changed lines of the file:
@@
 F 0 "C4" H 3960 2145 50  0000 L CNN
 F 1 "47uF" H 3960 1995 50  0000 L CNN
-F 2 "Resistors_SMD:R_1210" H 3950 2075 50  0001 C CNN
+F 2 "Capacitors_SMD:C_1210" H 3950 2075 50  0001 C CNN
 F 3 "" H 3950 2075 50  0001 C CNN
 F 4 "Murata" H 3950 2075 60  0001 C CNN "Manufacturer"
@@
 $EndComp
 $Comp
-L +12V #PWR06
+L +12V #PWR12
 U 1 1 568AC408
 P 5150 1925
-F 0 "#PWR06" H 5150 1775 50  0001 C CNN
+F 0 "#PWR12" H 5150 1775 50  0001 C CNN
 F 1 "+12V" H 5168 2099 50  0000 C CNN
 F 2 "" H 5150 1925 50  0000 C CNN
@@
 $EndComp
 $Comp
-L GND #PWR07
+L GND #PWR6
 U 1 1 568AE875
 P 1425 4450
-F 0 "#PWR07" H 1425 4200 50  0001 C CNN
+F 0 "#PWR6" H 1425 4200 50  0001 C CNN
 F 1 "GND" H 1433 4276 50  0000 C CNN
 F 2 "" H 1425 4450 50  0000 C CNN
@@
 $EndComp
 $Comp
-L GND #PWR08
+L GND #PWR11
 U 1 1 568AE8A5
 P 2800 2325
-F 0 "#PWR08" H 2800 2075 50  0001 C CNN
+F 0 "#PWR11" H 2800 2075 50  0001 C CNN
 F 1 "GND" H 2808 2151 50  0000 C CNN
 F 2 "" H 2800 2325 50  0000 C CNN
@@
 	1500 4350 1425 4350
 $Comp
-L Vsupply #P09
+L Vsupply #P5
 U 1 1 568AD53F
 P 4750 1225
-F 0 "#P09" H 4750 1225 60  0001 C CNN
+F 0 "#P5" H 4750 1225 60  0001 C CNN
 F 1 "Vsupply" H 4750 1175 34  0000 C CNN
 F 2 "" H 4750 1225 60  0000 C CNN
@@
 $EndComp
 $Comp
-L Vsupply #P010
+L Vsupply #P1
 U 1 1 568AD70E
 P 1525 1775
-F 0 "#P010" H 1525 1775 60  0001 C CNN
+F 0 "#P1" H 1525 1775 60  0001 C CNN
 F 1 "Vsupply" H 1525 1725 34  0000 C CNN
 F 2 "" H 1525 1775 60  0000 C CNN
@@
 $EndComp
 $Comp
-L GND #PWR011
+L GND #PWR7
 U 1 1 568ADBA9
 P 1450 3800
-F 0 "#PWR011" H 1450 3550 50  0001 C CNN
+F 0 "#PWR7" H 1450 3550 50  0001 C CNN
 F 1 "GND" H 1458 3626 50  0000 C CNN
 F 2 "" H 1450 3800 50  0000 C CNN
@@
 	1525 3700 1450 3700
 $Comp
-L Vsupply #P012
+L Vsupply #P4
 U 1 1 568ADC9C
 P 2125 3550
-F 0 "#P012" H 2125 3550 60  0001 C CNN
+F 0 "#P4" H 2125 3550 60  0001 C CNN
 F 1 "Vsupply" H 2125 3500 34  0000 C CNN
 F 2 "" H 2125 3550 60  0000 C CNN
@@
 $EndComp
 $Comp
-L Vheatbed #P013
+L Vheatbed #P3
 U 1 1 568AE31D
 P 2100 4200
-F 0 "#P013" H 2100 4200 60  0001 C CNN
+F 0 "#P3" H 2100 4200 60  0001 C CNN
 F 1 "Vheatbed" H 2100 4150 34  0000 C CNN
 F 2 "" H 2100 4200 60  0000 C CNN
@@
 $EndComp
 $Comp
-L GND #PWR014
+L GND #PWR8
 U 1 1 568AE68D
 P 1475 5400
-F 0 "#PWR014" H 1475 5150 50  0001 C CNN
+F 0 "#PWR8" H 1475 5150 50  0001 C CNN
 F 1 "GND" H 1483 5226 50  0000 C CNN
 F 2 "" H 1475 5400 50  0000 C CNN
@@
 	1475 5300 1650 5300
 $Comp
-L Vsupply #P015
+L Vsupply #P2
 U 1 1 568AE69B
 P 1650 5150
-F 0 "#P015" H 1650 5150 60  0001 C CNN
+F 0 "#P2" H 1650 5150 60  0001 C CNN
 F 1 "Vsupply" H 1650 5100 34  0000 C CNN
 F 2 "" H 1650 5150 60  0000 C CNN
@@
 $EndComp
 $Comp
-L GND #PWR016
+L GND #PWR9
 U 1 1 568AE860
 P 1475 6475
-F 0 "#PWR016" H 1475 6225 50  0001 C CNN
+F 0 "#PWR9" H 1475 6225 50  0001 C CNN
 F 1 "GND" H 1483 6301 50  0000 C CNN
 F 2 "" H 1475 6475 50  0000 C CNN
@@
 	1475 6375 1650 6375
 $Comp
-L +12V #PWR017
+L +12V #PWR10
 U 1 1 568BD457
 P 1650 6375
-F 0 "#PWR017" H 1650 6225 50  0001 C CNN
+F 0 "#PWR10" H 1650 6225 50  0001 C CNN
 F 1 "+12V" H 1668 6549 50  0000 C CNN
 F 2 "" H 1650 6375 50  0000 C CNN

Commit message: More 3d stuff
Parts:
- C1, C2: footprint Capacitors_SMD:C_0805 -> capacitors:C_0805
- C3: footprint Capacitors_SMD:C_0603 -> capacitors:C_0603
- D1: footprint armin-footprints:DO214AA -> diodes:DO214AA_SMB
- D2: footprint armin-footprints:DO214AC -> diodes:DO214AC_SMA
- F1, F2: footprint armin-footprints:FUSEHOLDER_MINI_KEYSTONE_3557 -> misc:FUSEHOLDER_MINI_KEYSTONE_3557
- P1, P2: footprint armin-footprints:CON_PHOENIX_MSTBA-2.5-2-G-5.08 -> terminal_blocks:CON_PHOENIX_MSTBA-2.5-2-G-5.08
- R2, R3: footprint Resistors_SMD:R_0603 -> resistors:R_0603
- U1: footprint armin-footprints:SOIC8 -> soic:SOIC8
Changed lines of the file:
@@
 F 0 "U1" H 2425 2475 34  0000 C BNN
 F 1 "MC34063" H 2425 2150 34  0000 C BNN
-F 2 "armin-footprints:SOIC8" H 2025 2100 60  0001 C CNN
+F 2 "soic:SOIC8" H 2025 2100 60  0001 C CNN
 F 3 "" H 2025 2100 60  0000 C CNN
 	1    2025 2100
@@
 F 0 "D1" H 3450 2100 34  0000 L BNN
 F 1 "STPS3L40UF" H 3375 2300 34  0000 L BNN
-F 2 "armin-footprints:DO214AA" H 3425 2175 60  0001 C CNN
+F 2 "diodes:DO214AA_SMB" H 3425 2175 60  0001 C CNN
 F 3 "" H 3425 2175 60  0000 C CNN
 	1    3425 2175
@@
 F 0 "C3" H 3035 2095 50  0000 L CNN
 F 1 "220pF" H 2825 1950 50  0000 L CNN
-F 2 "Capacitors_SMD:C_0603" H 3025 2025 50  0001 C CNN
+F 2 "capacitors:C_0603" H 3025 2025 50  0001 C CNN
 F 3 "" H 3025 2025 50  0000 C CNN
 	1    3025 2025
@@
 F 0 "R2" V 3875 1750 34  0000 L BNN
 F 1 "10K" H 3825 1900 34  0000 L BNN
-F 2 "Resistors_SMD:R_0603" H 3725 1825 60  0001 C CNN
+F 2 "resistors:R_0603" H 3725 1825 60  0001 C CNN
 F 3 "" H 3725 1825 60  0000 C CNN
 	1    3725 1825
@@
 F 0 "R3" V 3875 2175 34  0000 L BNN
 F 1 "1K1" H 3800 2050 34  0000 L BNN
-F 2 "Resistors_SMD:R_0603" H 3725 2100 60  0001 C CNN
+F 2 "resistors:R_0603" H 3725 2100 60  0001 C CNN
 F 3 "" H 3725 2100 60  0000 C CNN
 	1    3725 2100
@@
 F 0 "C1" H 1535 2145 50  0000 L CNN
 F 1 "10uF" H 1535 1995 50  0000 L CNN
-F 2 "Capacitors_SMD:C_0805" H 1525 2075 50  0001 C CNN
+F 2 "capacitors:C_0805" H 1525 2075 50  0001 C CNN
 F 3 "" H 1525 2075 50  0000 C CNN
 	1    1525 2075
@@
 F 0 "C2" H 1760 2145 50  0000 L CNN
 F 1 "10uF" H 1760 1995 50  0000 L CNN
-F 2 "Capacitors_SMD:C_0805" H 1750 2075 50  0001 C CNN
+F 2 "capacitors:C_0805" H 1750 2075 50  0001 C CNN
 F 3 "" H 1750 2075 50  0000 C CNN
 	1    1750 2075
@@
 F 0 "D2" H 4862 2907 34  0000 C CNN
 F 1 "ES1G" H 4862 2838 34  0000 C CNN
-F 2 "armin-footprints:DO214AC" H 4750 2675 60  0001 C CNN
+F 2 "diodes:DO214AC_SMA" H 4750 2675 60  0001 C CNN
 F 3 "" H 4750 2675 60  0000 C CNN
 	1    4750 2675
@@
 $EndComp
 $Comp
-L +12V #PWR12
+L +12V #PWR06
 U 1 1 568AC408
 P 5150 1925
-F 0 "#PWR12" H 5150 1775 50  0001 C CNN
+F 0 "#PWR06" H 5150 1775 50  0001 C CNN
 F 1 "+12V" H 5168 2099 50  0000 C CNN
 F 2 "" H 5150 1925 50  0000 C CNN
@@
 F 0 "P1" H 1250 4225 50  0000 C CNN
 F 1 "CONN_01X02" H 1144 4210 50  0001 C CNN
-F 2 "armin-footprints:CON_PHOENIX_MSTBA-2.5-2-G-5.08" H 1225 4400 50  0001 C CNN
+F 2 "terminal_blocks:CON_PHOENIX_MSTBA-2.5-2-G-5.08" H 1225 4400 50  0001 C CNN
 F 3 "" H 1225 4400 50  0000 C CNN
 	1    1225 4400
@@
 $EndComp
 $Comp
-L GND #PWR6
+L GND #PWR07
 U 1 1 568AE875
 P 1425 4450
-F 0 "#PWR6" H 1425 4200 50  0001 C CNN
+F 0 "#PWR07" H 1425 4200 50  0001 C CNN
 F 1 "GND" H 1433 4276 50  0000 C CNN
 F 2 "" H 1425 4450 50  0000 C CNN
@@
 $EndComp
 $Comp
-L GND #PWR11
+L GND #PWR08
 U 1 1 568AE8A5
 P 2800 2325
-F 0 "#PWR11" H 2800 2075 50  0001 C CNN
+F 0 "#PWR08" H 2800 2075 50  0001 C CNN
 F 1 "GND" H 2808 2151 50  0000 C CNN
 F 2 "" H 2800 2325 50  0000 C CNN
@@
 F 0 "F1" H 1750 4591 50  0000 C CNN
 F 1 "FUSE" H 1750 4499 50  0000 C CNN
-F 2 "armin-footprints:FUSEHOLDER_MINI_KEYSTONE_3557" H 1750 4350 50  0001 C CNN
+F 2 "misc:FUSEHOLDER_MINI_KEYSTONE_3557" H 1750 4350 50  0001 C CNN
 F 3 "" H 1750 4350 50  0000 C CNN
 	1    1750 4350
@@
 	1500 4350 1425 4350
 $Comp
-L Vsupply #P5
+L Vsupply #P09
 U 1 1 568AD53F
 P 4750 1225
-F 0 "#P5" H 4750 1225 60  0001 C CNN
+F 0 "#P09" H 4750 1225 60  0001 C CNN
 F 1 "Vsupply" H 4750 1175 34  0000 C CNN
 F 2 "" H 4750 1225 60  0000 C CNN
@@
 $EndComp
 $Comp
-L Vsupply #P1
+L Vsupply #P010
 U 1 1 568AD70E
 P 1525 1775
-F 0 "#P1" H 1525 1775 60  0001 C CNN
+F 0 "#P010" H 1525 1775 60  0001 C CNN
 F 1 "Vsupply" H 1525 1725 34  0000 C CNN
 F 2 "" H 1525 1775 60  0000 C CNN
@@
 F 0 "P2" H 1250 3575 50  0000 C CNN
 F 1 "CONN_01X02" H 1169 3560 50  0001 C CNN
-F 2 "armin-footprints:CON_PHOENIX_MSTBA-2.5-2-G-5.08" H 1250 3750 50  0001 C CNN
+F 2 "terminal_blocks:CON_PHOENIX_MSTBA-2.5-2-G-5.08" H 1250 3750 50  0001 C CNN
 F 3 "" H 1250 3750 50  0000 C CNN
 	1    1250 3750
@@
 $EndComp
 $Comp
-L GND #PWR7
+L GND #PWR011
 U 1 1 568ADBA9
 P 1450 3800
-F 0 "#PWR7" H 1450 3550 50  0001 C CNN
+F 0 "#PWR011" H 1450 3550 50  0001 C CNN
 F 1 "GND" H 1458 3626 50  0000 C CNN
 F 2 "" H 1450 3800 50  0000 C CNN
@@
 F 0 "F2" H 1775 3941 50  0000 C CNN
 F 1 "FUSE" H 1775 3849 50  0000 C CNN
-F 2 "armin-footprints:FUSEHOLDER_MINI_KEYSTONE_3557" H 1775 3700 50  0001 C CNN
+F 2 "misc:FUSEHOLDER_MINI_KEYSTONE_3557" H 1775 3700 50  0001 C CNN
 F 3 "" H 1775 3700 50  0000 C CNN
 	1    1775 3700
@@
 	1525 3700 1450 3700
 $Comp
-L Vsupply #P4
+L Vsupply #P012
 U 1 1 568ADC9C
 P 2125 3550
-F 0 "#P4" H 2125 3550 60  0001 C CNN
+F 0 "#P012" H 2125 3550 60  0001 C CNN
 F 1 "Vsupply" H 2125 3500 34  0000 C CNN
 F 2 "" H 2125 3550 60  0000 C CNN
@@
 $EndComp
 $Comp
-L Vheatbed #P3
+L Vheatbed #P013
 U 1 1 568AE31D
 P 2100 4200
-F 0 "#P3" H 2100 4200 60  0001 C CNN
+F 0 "#P013" H 2100 4200 60  0001 C CNN
 F 1 "Vheatbed" H 2100 4150 34  0000 C CNN
 F 2 "" H 2100 4200 60  0000 C CNN
@@
 $EndComp
 $Comp
-L GND #PWR8
+L GND #PWR014
 U 1 1 568AE68D
 P 1475 5400
-F 0 "#PWR8" H 1475 5150 50  0001 C CNN
+F 0 "#PWR014" H 1475 5150 50  0001 C CNN
 F 1 "GND" H 1483 5226 50  0000 C CNN
 F 2 "" H 1475 5400 50  0000 C CNN
@@
 	1475 5300 1650 5300
 $Comp
-L Vsupply #P2
+L Vsupply #P015
 U 1 1 568AE69B
 P 1650 5150
-F 0 "#P2" H 1650 5150 60  0001 C CNN
+F 0 "#P015" H 1650 5150 60  0001 C CNN
 F 1 "Vsupply" H 1650 5100 34  0000 C CNN
 F 2 "" H 1650 5150 60  0000 C CNN
@@
 $EndComp
 $Comp
-L GND #PWR9
+L GND #PWR016
 U 1 1 568AE860
 P 1475 6475
-F 0 "#PWR9" H 1475 6225 50  0001 C CNN
+F 0 "#PWR016" H 1475 6225 50  0001 C CNN
 F 1 "GND" H 1483 6301 50  0000 C CNN
 F 2 "" H 1475 6475 50  0000 C CNN
@@
 	1475 6375 1650 6375
 $Comp
-L +12V #PWR10
+L +12V #PWR017
 U 1 1 568BD457
 P 1650 6375
-F 0 "#PWR10" H 1650 6225 50  0001 C CNN
+F 0 "#PWR017" H 1650 6225 50  0001 C CNN
 F 1 "+12V" H 1668 6549 50  0000 C CNN
 F 2 "" H 1650 6375 50  0000 C CNN

Commit message: cleanup
Parts:
- C4: footprint Capacitors_SMD:C_1210 -> capacitors:C_1210
- L1: footprint armin-footprints:INDUCTOR_AIUR06 -> inductors:INDUCTOR_AIUR06
- R1: footprint Resistors_SMD:R_1206 -> resistors:R_1206
Changed lines of the file:
@@
 F 0 "L1" V 3650 1800 50  0000 L CNN
 F 1 "100uH" V 3525 1725 50  0000 L CNN
-F 2 "armin-footprints:INDUCTOR_AIUR06" H 3575 1825 50  0001 C CNN
+F 2 "inductors:INDUCTOR_AIUR06" H 3575 1825 50  0001 C CNN
 F 3 "" H 3575 1825 50  0000 C CNN
 	1    3575 1825
@@
 F 0 "C4" H 3960 2145 50  0000 L CNN
 F 1 "47uF" H 3960 1995 50  0000 L CNN
-F 2 "Capacitors_SMD:C_1210" H 3950 2075 50  0001 C CNN
+F 2 "capacitors:C_1210" H 3950 2075 50  0001 C CNN
 F 3 "" H 3950 2075 50  0001 C CNN
 F 4 "Murata" H 3950 2075 60  0001 C CNN "Manufacturer"
@@
 F 0 "R1" H 1850 1900 34  0000 L BNN
 F 1 "0.22R" H 1800 1800 34  0000 L BNN
-F 2 "Resistors_SMD:R_1206" H 1750 1850 60  0001 C CNN
+F 2 "resistors:R_1206" H 1750 1850 60  0001 C CNN
 F 3 "" H 1750 1850 60  0000 C CNN
 	1    1750 1850

Commit message: fixed minor issue
Parts:
- JP1: footprint armin-footprints:CON_HDR_1x3_2.54mm -> headers:CON_HDR_1x3_2.54mm
- JP2, P3, P4: footprint armin-footprints:CON_HDR_1x2_2.54mm -> headers:CON_HDR_1x2_2.54mm
Changed lines of the file:
@@
 F 0 "JP1" H 4400 2065 50  0000 C CNN
 F 1 "VSEL" H 4400 1973 50  0000 C CNN
-F 2 "armin-footprints:CON_HDR_1x3_2.54mm" H 4400 1825 50  0001 C CNN
+F 2 "headers:CON_HDR_1x3_2.54mm" H 4400 1825 50  0001 C CNN
 F 3 "" H 4400 1825 50  0000 C CNN
 	1    4400 1825
@@
 F 0 "JP2" H 5850 2890 50  0000 C CNN
 F 1 "BOARD_POWER" H 5850 2798 50  0000 C CNN
-F 2 "armin-footprints:CON_HDR_1x2_2.54mm" H 5850 2625 50  0001 C CNN
+F 2 "headers:CON_HDR_1x2_2.54mm" H 5850 2625 50  0001 C CNN
 F 3 "" H 5850 2625 50  0000 C CNN
 	1    5850 2625
@@
 F 0 "P3" H 1275 5175 50  0000 C CNN
 F 1 "CONN_01X02" H 1194 5160 50  0001 C CNN
-F 2 "armin-footprints:CON_HDR_1x2_2.54mm" H 1275 5350 50  0001 C CNN
+F 2 "headers:CON_HDR_1x2_2.54mm" H 1275 5350 50  0001 C CNN
 F 3 "" H 1275 5350 50  0000 C CNN
 	1    1275 5350
@@
 F 0 "P4" H 1275 6250 50  0000 C CNN
 F 1 "CONN_01X02" H 1194 6235 50  0001 C CNN
-F 2 "armin-footprints:CON_HDR_1x2_2.54mm" H 1275 6425 50  0001 C CNN
+F 2 "headers:CON_HDR_1x2_2.54mm" H 1275 6425 50  0001 C CNN
 F 3 "" H 1275 6425 50  0000 C CNN
 	1    1275 6425
