File: steppers.sch (KiCad schematic (older format))
At the start: 24 parts, among them J1 HEADER, J10 STEPSTICK, J11 STEPSTICK, J12 STEPSTICK, J2 HEADER, J3 HEADER, J4 STEPSTICK, J5 STEPSTICK, J6 STEPSTICK, J7 HEADER, J8 HEADER, J9 HEADER, P10 CONN_01X04, P11 CONN_01X04, P12 CONN_01X04, P7 CONN_02X04, P8 CONN_01X04, P9 CONN_01X04

Commit message: Added 3d models
Parts:
- J1, J2, J3, J7, J8, J9: footprint geda-footprints:CON_HDR_2x3 -> armin-footprints:CON_HDR_2x3_2.54mm
- P10, P11, P12, P8, P9: footprint geda-footprints:CON_HDR_1x4 -> armin-footprints:CON_HDR_1x4_2.54mm
- P7: footprint geda-footprints:CON_HDR_2x4 -> armin-footprints:CON_HDR_2x4_2.54mm
Changed lines of the file:
@@
 F 0 "J2" H 1675 1907 34  0000 C CNN
 F 1 "HEADER" H 1675 1838 34  0000 C CNN
-F 2 "geda-footprints:CON_HDR_2x3" H 1500 1475 60  0001 C CNN
+F 2 "armin-footprints:CON_HDR_2x3_2.54mm" H 1500 1475 60  0001 C CNN
 F 3 "" H 1500 1475 60  0000 C CNN
 	1    1500 1475
@@
 F 0 "P8" H 3477 1513 50  0000 L CNN
 F 1 "CONN_01X04" H 3477 1421 50  0000 L CNN
-F 2 "geda-footprints:CON_HDR_1x4" H 3400 1475 50  0001 C CNN
+F 2 "armin-footprints:CON_HDR_1x4_2.54mm" H 3400 1475 50  0001 C CNN
 F 3 "" H 3400 1475 50  0000 C CNN
 	1    3400 1475
@@
 F 0 "J3" H 1675 3132 34  0000 C CNN
 F 1 "HEADER" H 1675 3063 34  0000 C CNN
-F 2 "geda-footprints:CON_HDR_2x3" H 1500 2700 60  0001 C CNN
+F 2 "armin-footprints:CON_HDR_2x3_2.54mm" H 1500 2700 60  0001 C CNN
 F 3 "" H 1500 2700 60  0000 C CNN
 	1    1500 2700
@@
 F 0 "P9" H 3477 2738 50  0000 L CNN
 F 1 "CONN_01X04" H 3477 2646 50  0000 L CNN
-F 2 "geda-footprints:CON_HDR_1x4" H 3400 2700 50  0001 C CNN
+F 2 "armin-footprints:CON_HDR_1x4_2.54mm" H 3400 2700 50  0001 C CNN
 F 3 "" H 3400 2700 50  0000 C CNN
 	1    3400 2700
@@
 F 0 "J7" H 6775 4557 34  0000 C CNN
 F 1 "HEADER" H 6775 4488 34  0000 C CNN
-F 2 "geda-footprints:CON_HDR_2x3" H 6600 4125 60  0001 C CNN
+F 2 "armin-footprints:CON_HDR_2x3_2.54mm" H 6600 4125 60  0001 C CNN
 F 3 "" H 6600 4125 60  0000 C CNN
 	1    6600 4125
@@
 F 0 "P10" H 8577 4163 50  0000 L CNN
 F 1 "CONN_01X04" H 8577 4071 50  0000 L CNN
-F 2 "geda-footprints:CON_HDR_1x4" H 8500 4125 50  0001 C CNN
+F 2 "armin-footprints:CON_HDR_1x4_2.54mm" H 8500 4125 50  0001 C CNN
 F 3 "" H 8500 4125 50  0000 C CNN
 	1    8500 4125
@@
 F 0 "J8" H 6750 1882 34  0000 C CNN
 F 1 "HEADER" H 6750 1813 34  0000 C CNN
-F 2 "geda-footprints:CON_HDR_2x3" H 6575 1450 60  0001 C CNN
+F 2 "armin-footprints:CON_HDR_2x3_2.54mm" H 6575 1450 60  0001 C CNN
 F 3 "" H 6575 1450 60  0000 C CNN
 	1    6575 1450
@@
 F 0 "P11" H 8552 1488 50  0000 L CNN
 F 1 "CONN_01X04" H 8552 1396 50  0000 L CNN
-F 2 "geda-footprints:CON_HDR_1x4" H 8475 1450 50  0001 C CNN
+F 2 "armin-footprints:CON_HDR_1x4_2.54mm" H 8475 1450 50  0001 C CNN
 F 3 "" H 8475 1450 50  0000 C CNN
 	1    8475 1450
@@
 F 0 "J9" H 6750 3257 34  0000 C CNN
 F 1 "HEADER" H 6750 3188 34  0000 C CNN
-F 2 "geda-footprints:CON_HDR_2x3" H 6575 2825 60  0001 C CNN
+F 2 "armin-footprints:CON_HDR_2x3_2.54mm" H 6575 2825 60  0001 C CNN
 F 3 "" H 6575 2825 60  0000 C CNN
 	1    6575 2825
@@
 F 0 "P12" H 8552 2863 50  0000 L CNN
 F 1 "CONN_01X04" H 8552 2771 50  0000 L CNN
-F 2 "geda-footprints:CON_HDR_1x4" H 8475 2825 50  0001 C CNN
+F 2 "armin-footprints:CON_HDR_1x4_2.54mm" H 8475 2825 50  0001 C CNN
 F 3 "" H 8475 2825 50  0000 C CNN
 	1    8475 2825
@@
 F 0 "P7" H 3425 4250 50  0000 C CNN
 F 1 "CONN_02X04" H 3425 3750 50  0000 C CNN
-F 2 "geda-footprints:CON_HDR_2x4" H 3425 2800 50  0001 C CNN
+F 2 "armin-footprints:CON_HDR_2x4_2.54mm" H 3425 2800 50  0001 C CNN
 F 3 "" H 3425 2800 50  0000 C CNN
 	1    3425 4000
@@
 F 0 "J1" H 1650 4432 34  0000 C CNN
 F 1 "HEADER" H 1650 4363 34  0000 C CNN
-F 2 "geda-footprints:CON_HDR_2x3" H 1475 4000 60  0001 C CNN
+F 2 "armin-footprints:CON_HDR_2x3_2.54mm" H 1475 4000 60  0001 C CNN
 F 3 "" H 1475 4000 60  0000 C CNN
 	1    1475 4000

Commit message: More 3d stuff
Parts:
- J10, J11, J12, J4, J5, J6: footprint geda-footprints:STEPSTICK -> armin-footprints:STEPSTICK
Changed lines of the file:
@@
 F 0 "J5" H 2475 2750 34  0000 C CNN
 F 1 "STEPSTICK" H 2475 2650 34  0000 C CNN
-F 2 "geda-footprints:STEPSTICK" H 2025 1925 60  0001 C CNN
+F 2 "armin-footprints:STEPSTICK" H 2025 1925 60  0001 C CNN
 F 3 "" H 2025 1925 60  0000 C CNN
 	1    2025 1925
@@
 $EndComp
 $Comp
-L Vsupply #P053
+L Vsupply #P17
 U 1 1 568BEEB3
 P 3150 775
-F 0 "#P053" H 3150 775 60  0001 C CNN
+F 0 "#P17" H 3150 775 60  0001 C CNN
 F 1 "Vsupply" H 3150 725 34  0000 C CNN
 F 2 "" H 3150 775 60  0000 C CNN
@@
 	1150 1125 1150 1425
 $Comp
-L +3.3V #PWR054
+L +3.3V #PWR39
 U 1 1 568BF4F0
 P 1150 1125
-F 0 "#PWR054" H 1150 975 50  0001 C CNN
+F 0 "#PWR39" H 1150 975 50  0001 C CNN
 F 1 "+3.3V" H 1168 1299 50  0000 C CNN
 F 2 "" H 1150 1125 50  0000 C CNN
@@
 $EndComp
 $Comp
-L +3.3V #PWR055
+L +3.3V #PWR45
 U 1 1 568BFD7B
 P 3050 1725
-F 0 "#PWR055" H 3050 1575 50  0001 C CNN
+F 0 "#PWR45" H 3050 1575 50  0001 C CNN
 F 1 "+3.3V" H 3050 1850 50  0000 C CNN
 F 2 "" H 3050 1725 50  0000 C CNN
@@
 	2900 1725 3050 1725
 $Comp
-L GND #PWR056
+L GND #PWR42
 U 1 1 568BFE54
 P 2975 1225
-F 0 "#PWR056" H 2975 975 50  0001 C CNN
+F 0 "#PWR42" H 2975 975 50  0001 C CNN
 F 1 "GND" H 2983 1051 50  0000 C CNN
 F 2 "" H 2975 1225 50  0000 C CNN
@@
 $EndComp
 $Comp
-L GND #PWR057
+L GND #PWR48
 U 1 1 568BFE70
 P 3225 1825
-F 0 "#PWR057" H 3225 1575 50  0001 C CNN
+F 0 "#PWR48" H 3225 1575 50  0001 C CNN
 F 1 "GND" H 3233 1651 50  0000 C CNN
 F 2 "" H 3225 1825 50  0000 C CNN
@@
 F 0 "J6" H 2475 3975 34  0000 C CNN
 F 1 "STEPSTICK" H 2475 3875 34  0000 C CNN
-F 2 "geda-footprints:STEPSTICK" H 2025 3150 60  0001 C CNN
+F 2 "armin-footprints:STEPSTICK" H 2025 3150 60  0001 C CNN
 F 3 "" H 2025 3150 60  0000 C CNN
 	1    2025 3150
@@
 $EndComp
 $Comp
-L Vsupply #P058
+L Vsupply #P18
 U 1 1 568BD851
 P 3150 2000
-F 0 "#P058" H 3150 2000 60  0001 C CNN
+F 0 "#P18" H 3150 2000 60  0001 C CNN
 F 1 "Vsupply" H 3150 1950 34  0000 C CNN
 F 2 "" H 3150 2000 60  0000 C CNN
@@
 	1150 2375 1150 2650
 $Comp
-L +3.3V #PWR059
+L +3.3V #PWR40
 U 1 1 568BD862
 P 1150 2375
-F 0 "#PWR059" H 1150 2225 50  0001 C CNN
+F 0 "#PWR40" H 1150 2225 50  0001 C CNN
 F 1 "+3.3V" H 1168 2549 50  0000 C CNN
 F 2 "" H 1150 2375 50  0000 C CNN
@@
 $EndComp
 $Comp
-L +3.3V #PWR060
+L +3.3V #PWR46
 U 1 1 568BD86E
 P 3050 2950
-F 0 "#PWR060" H 3050 2800 50  0001 C CNN
+F 0 "#PWR46" H 3050 2800 50  0001 C CNN
 F 1 "+3.3V" H 3050 3075 50  0000 C CNN
 F 2 "" H 3050 2950 50  0000 C CNN
@@
 	2900 2950 3050 2950
 $Comp
-L GND #PWR061
+L GND #PWR43
 U 1 1 568BD875
 P 2975 2450
-F 0 "#PWR061" H 2975 2200 50  0001 C CNN
+F 0 "#PWR43" H 2975 2200 50  0001 C CNN
 F 1 "GND" H 2983 2276 50  0000 C CNN
 F 2 "" H 2975 2450 50  0000 C CNN
@@
 $EndComp
 $Comp
-L GND #PWR062
+L GND #PWR49
 U 1 1 568BD87B
 P 3225 3050
-F 0 "#PWR062" H 3225 2800 50  0001 C CNN
+F 0 "#PWR49" H 3225 2800 50  0001 C CNN
 F 1 "GND" H 3233 2876 50  0000 C CNN
 F 2 "" H 3225 3050 50  0000 C CNN
@@
 F 0 "J4" H 2450 5275 34  0000 C CNN
 F 1 "STEPSTICK" H 2450 5175 34  0000 C CNN
-F 2 "geda-footprints:STEPSTICK" H 2000 4450 60  0001 C CNN
+F 2 "armin-footprints:STEPSTICK" H 2000 4450 60  0001 C CNN
 F 3 "" H 2000 4450 60  0000 C CNN
 	1    2000 4450
@@
 $EndComp
 $Comp
-L Vsupply #P063
+L Vsupply #P16
 U 1 1 568BDFCA
 P 3125 3300
-F 0 "#P063" H 3125 3300 60  0001 C CNN
+F 0 "#P16" H 3125 3300 60  0001 C CNN
 F 1 "Vsupply" H 3125 3250 34  0000 C CNN
 F 2 "" H 3125 3300 60  0000 C CNN
@@
 	1125 3650 1125 3950
 $Comp
-L +3.3V #PWR064
+L +3.3V #PWR38
 U 1 1 568BDFDB
 P 1125 3650
-F 0 "#PWR064" H 1125 3500 50  0001 C CNN
+F 0 "#PWR38" H 1125 3500 50  0001 C CNN
 F 1 "+3.3V" H 1143 3824 50  0000 C CNN
 F 2 "" H 1125 3650 50  0000 C CNN
@@
 $EndComp
 $Comp
-L +3.3V #PWR065
+L +3.3V #PWR44
 U 1 1 568BDFE7
 P 3025 4250
-F 0 "#PWR065" H 3025 4100 50  0001 C CNN
+F 0 "#PWR44" H 3025 4100 50  0001 C CNN
 F 1 "+3.3V" H 3025 4375 50  0000 C CNN
 F 2 "" H 3025 4250 50  0000 C CNN
@@
 	2875 4250 3025 4250
 $Comp
-L GND #PWR066
+L GND #PWR41
 U 1 1 568BDFEE
 P 2950 3750
-F 0 "#PWR066" H 2950 3500 50  0001 C CNN
+F 0 "#PWR41" H 2950 3500 50  0001 C CNN
 F 1 "GND" H 2958 3576 50  0000 C CNN
 F 2 "" H 2950 3750 50  0000 C CNN
@@
 $EndComp
 $Comp
-L GND #PWR067
+L GND #PWR47
 U 1 1 568BDFF4
 P 3200 4350
-F 0 "#PWR067" H 3200 4100 50  0001 C CNN
+F 0 "#PWR47" H 3200 4100 50  0001 C CNN
 F 1 "GND" H 3208 4176 50  0000 C CNN
 F 2 "" H 3200 4350 50  0000 C CNN
@@
 F 0 "J10" H 7575 5400 34  0000 C CNN
 F 1 "STEPSTICK" H 7575 5300 34  0000 C CNN
-F 2 "geda-footprints:STEPSTICK" H 7125 4575 60  0001 C CNN
+F 2 "armin-footprints:STEPSTICK" H 7125 4575 60  0001 C CNN
 F 3 "" H 7125 4575 60  0000 C CNN
 	1    7125 4575
@@
 $EndComp
 $Comp
-L Vsupply #P068
+L Vsupply #P21
 U 1 1 568C39F8
 P 8250 3425
-F 0 "#P068" H 8250 3425 60  0001 C CNN
+F 0 "#P21" H 8250 3425 60  0001 C CNN
 F 1 "Vsupply" H 8250 3375 34  0000 C CNN
 F 2 "" H 8250 3425 60  0000 C CNN
@@
 	6250 4075 6250 3775
 $Comp
-L +3.3V #PWR069
+L +3.3V #PWR52
 U 1 1 568C3A09
 P 6250 3775
-F 0 "#PWR069" H 6250 3625 50  0001 C CNN
+F 0 "#PWR52" H 6250 3625 50  0001 C CNN
 F 1 "+3.3V" H 6268 3949 50  0000 C CNN
 F 2 "" H 6250 3775 50  0000 C CNN
@@
 $EndComp
 $Comp
-L +3.3V #PWR070
+L +3.3V #PWR58
 U 1 1 568C3A15
 P 8150 4375
-F 0 "#PWR070" H 8150 4225 50  0001 C CNN
+F 0 "#PWR58" H 8150 4225 50  0001 C CNN
 F 1 "+3.3V" H 8150 4500 50  0000 C CNN
 F 2 "" H 8150 4375 50  0000 C CNN
@@
 	8000 4375 8150 4375
 $Comp
-L GND #PWR071
+L GND #PWR55
 U 1 1 568C3A1C
 P 8075 3875
-F 0 "#PWR071" H 8075 3625 50  0001 C CNN
+F 0 "#PWR55" H 8075 3625 50  0001 C CNN
 F 1 "GND" H 8083 3701 50  0000 C CNN
 F 2 "" H 8075 3875 50  0000 C CNN
@@
 $EndComp
 $Comp
-L GND #PWR072
+L GND #PWR61
 U 1 1 568C3A22
 P 8325 4475
-F 0 "#PWR072" H 8325 4225 50  0001 C CNN
+F 0 "#PWR61" H 8325 4225 50  0001 C CNN
 F 1 "GND" H 8333 4301 50  0000 C CNN
 F 2 "" H 8325 4475 50  0000 C CNN
@@
 F 0 "J11" H 7550 2725 34  0000 C CNN
 F 1 "STEPSTICK" H 7550 2625 34  0000 C CNN
-F 2 "geda-footprints:STEPSTICK" H 7100 1900 60  0001 C CNN
+F 2 "armin-footprints:STEPSTICK" H 7100 1900 60  0001 C CNN
 F 3 "" H 7100 1900 60  0000 C CNN
 	1    7100 1900
@@
 $EndComp
 $Comp
-L Vsupply #P073
+L Vsupply #P19
 U 1 1 568C3E5C
 P 8225 750
-F 0 "#P073" H 8225 750 60  0001 C CNN
+F 0 "#P19" H 8225 750 60  0001 C CNN
 F 1 "Vsupply" H 8225 700 34  0000 C CNN
 F 2 "" H 8225 750 60  0000 C CNN
@@
 	6225 1100 6225 1400
 $Comp
-L +3.3V #PWR074
+L +3.3V #PWR50
 U 1 1 568C3E6D
 P 6225 1100
-F 0 "#PWR074" H 6225 950 50  0001 C CNN
+F 0 "#PWR50" H 6225 950 50  0001 C CNN
 F 1 "+3.3V" H 6243 1274 50  0000 C CNN
 F 2 "" H 6225 1100 50  0000 C CNN
@@
 $EndComp
 $Comp
-L +3.3V #PWR075
+L +3.3V #PWR56
 U 1 1 568C3E79
 P 8125 1700
-F 0 "#PWR075" H 8125 1550 50  0001 C CNN
+F 0 "#PWR56" H 8125 1550 50  0001 C CNN
 F 1 "+3.3V" H 8125 1825 50  0000 C CNN
 F 2 "" H 8125 1700 50  0000 C CNN
@@
 	7975 1700 8125 1700
 $Comp
-L GND #PWR076
+L GND #PWR53
 U 1 1 568C3E80
 P 8050 1200
-F 0 "#PWR076" H 8050 950 50  0001 C CNN
+F 0 "#PWR53" H 8050 950 50  0001 C CNN
 F 1 "GND" H 8058 1026 50  0000 C CNN
 F 2 "" H 8050 1200 50  0000 C CNN
@@
 $EndComp
 $Comp
-L GND #PWR077
+L GND #PWR59
 U 1 1 568C3E86
 P 8300 1800
-F 0 "#PWR077" H 8300 1550 50  0001 C CNN
+F 0 "#PWR59" H 8300 1550 50  0001 C CNN
 F 1 "GND" H 8308 1626 50  0000 C CNN
 F 2 "" H 8300 1800 50  0000 C CNN
@@
 F 0 "J12" H 7550 4100 34  0000 C CNN
 F 1 "STEPSTICK" H 7550 4000 34  0000 C CNN
-F 2 "geda-footprints:STEPSTICK" H 7100 3275 60  0001 C CNN
+F 2 "armin-footprints:STEPSTICK" H 7100 3275 60  0001 C CNN
 F 3 "" H 7100 3275 60  0000 C CNN
 	1    7100 3275
@@
 $EndComp
 $Comp
-L Vsupply #P078
+L Vsupply #P20
 U 1 1 568C4325
 P 8225 2125
-F 0 "#P078" H 8225 2125 60  0001 C CNN
+F 0 "#P20" H 8225 2125 60  0001 C CNN
 F 1 "Vsupply" H 8225 2075 34  0000 C CNN
 F 2 "" H 8225 2125 60  0000 C CNN
@@
 	6225 2475 6225 2775
 $Comp
-L +3.3V #PWR079
+L +3.3V #PWR51
 U 1 1 568C4336
 P 6225 2475
-F 0 "#PWR079" H 6225 2325 50  0001 C CNN
+F 0 "#PWR51" H 6225 2325 50  0001 C CNN
 F 1 "+3.3V" H 6243 2649 50  0000 C CNN
 F 2 "" H 6225 2475 50  0000 C CNN
@@
 $EndComp
 $Comp
-L +3.3V #PWR080
+L +3.3V #PWR57
 U 1 1 568C4342
 P 8125 3075
-F 0 "#PWR080" H 8125 2925 50  0001 C CNN
+F 0 "#PWR57" H 8125 2925 50  0001 C CNN
 F 1 "+3.3V" H 8125 3200 50  0000 C CNN
 F 2 "" H 8125 3075 50  0000 C CNN
@@
 	7975 3075 8125 3075
 $Comp
-L GND #PWR081
+L GND #PWR54
 U 1 1 568C4349
 P 8050 2575
-F 0 "#PWR081" H 8050 2325 50  0001 C CNN
+F 0 "#PWR54" H 8050 2325 50  0001 C CNN
 F 1 "GND" H 8058 2401 50  0000 C CNN
 F 2 "" H 8050 2575 50  0000 C CNN
@@
 $EndComp
 $Comp
-L GND #PWR082
+L GND #PWR60
 U 1 1 568C434F
 P 8300 3175
-F 0 "#PWR082" H 8300 2925 50  0001 C CNN
+F 0 "#PWR60" H 8300 2925 50  0001 C CNN
 F 1 "GND" H 8308 3001 50  0000 C CNN
 F 2 "" H 8300 3175 50  0000 C CNN

Commit message: More 3d stuff
Parts:
- C12, C13, C14, C15, C16, C17: footprint armin-footprints:ELCO-8mm -> capacitors:ELCO-8mm-3.5mm_pitch
Changed lines of the file:
@@
 F 0 "C13" H 3888 1471 50  0000 L CNN
 F 1 "100uF" H 3888 1379 50  0000 L CNN
-F 2 "armin-footprints:ELCO-8mm" H 3800 1425 50  0001 C CNN
+F 2 "capacitors:ELCO-8mm-3.5mm_pitch" H 3800 1425 50  0001 C CNN
 F 3 "" H 3800 1425 50  0000 C CNN
 	1    3800 1425
@@
 $EndComp
 $Comp
-L Vsupply #P17
+L Vsupply #P053
 U 1 1 568BEEB3
 P 3150 775
-F 0 "#P17" H 3150 775 60  0001 C CNN
+F 0 "#P053" H 3150 775 60  0001 C CNN
 F 1 "Vsupply" H 3150 725 34  0000 C CNN
 F 2 "" H 3150 775 60  0000 C CNN
@@
 	1150 1125 1150 1425
 $Comp
-L +3.3V #PWR39
+L +3.3V #PWR054
 U 1 1 568BF4F0
 P 1150 1125
-F 0 "#PWR39" H 1150 975 50  0001 C CNN
+F 0 "#PWR054" H 1150 975 50  0001 C CNN
 F 1 "+3.3V" H 1168 1299 50  0000 C CNN
 F 2 "" H 1150 1125 50  0000 C CNN
@@
 $EndComp
 $Comp
-L +3.3V #PWR45
+L +3.3V #PWR055
 U 1 1 568BFD7B
 P 3050 1725
-F 0 "#PWR45" H 3050 1575 50  0001 C CNN
+F 0 "#PWR055" H 3050 1575 50  0001 C CNN
 F 1 "+3.3V" H 3050 1850 50  0000 C CNN
 F 2 "" H 3050 1725 50  0000 C CNN
@@
 	2900 1725 3050 1725
 $Comp
-L GND #PWR42
+L GND #PWR056
 U 1 1 568BFE54
 P 2975 1225
-F 0 "#PWR42" H 2975 975 50  0001 C CNN
+F 0 "#PWR056" H 2975 975 50  0001 C CNN
 F 1 "GND" H 2983 1051 50  0000 C CNN
 F 2 "" H 2975 1225 50  0000 C CNN
@@
 $EndComp
 $Comp
-L GND #PWR48
+L GND #PWR057
 U 1 1 568BFE70
 P 3225 1825
-F 0 "#PWR48" H 3225 1575 50  0001 C CNN
+F 0 "#PWR057" H 3225 1575 50  0001 C CNN
 F 1 "GND" H 3233 1651 50  0000 C CNN
 F 2 "" H 3225 1825 50  0000 C CNN
@@
 F 0 "C14" H 3888 2696 50  0000 L CNN
 F 1 "100uF" H 3888 2604 50  0000 L CNN
-F 2 "armin-footprints:ELCO-8mm" H 3800 2650 50  0001 C CNN
+F 2 "capacitors:ELCO-8mm-3.5mm_pitch" H 3800 2650 50  0001 C CNN
 F 3 "" H 3800 2650 50  0000 C CNN
 	1    3800 2650
@@
 $EndComp
 $Comp
-L Vsupply #P18
+L Vsupply #P058
 U 1 1 568BD851
 P 3150 2000
-F 0 "#P18" H 3150 2000 60  0001 C CNN
+F 0 "#P058" H 3150 2000 60  0001 C CNN
 F 1 "Vsupply" H 3150 1950 34  0000 C CNN
 F 2 "" H 3150 2000 60  0000 C CNN
@@
 	1150 2375 1150 2650
 $Comp
-L +3.3V #PWR40
+L +3.3V #PWR059
 U 1 1 568BD862
 P 1150 2375
-F 0 "#PWR40" H 1150 2225 50  0001 C CNN
+F 0 "#PWR059" H 1150 2225 50  0001 C CNN
 F 1 "+3.3V" H 1168 2549 50  0000 C CNN
 F 2 "" H 1150 2375 50  0000 C CNN
@@
 $EndComp
 $Comp
-L +3.3V #PWR46
+L +3.3V #PWR060
 U 1 1 568BD86E
 P 3050 2950
-F 0 "#PWR46" H 3050 2800 50  0001 C CNN
+F 0 "#PWR060" H 3050 2800 50  0001 C CNN
 F 1 "+3.3V" H 3050 3075 50  0000 C CNN
 F 2 "" H 3050 2950 50  0000 C CNN
@@
 	2900 2950 3050 2950
 $Comp
-L GND #PWR43
+L GND #PWR061
 U 1 1 568BD875
 P 2975 2450
-F 0 "#PWR43" H 2975 2200 50  0001 C CNN
+F 0 "#PWR061" H 2975 2200 50  0001 C CNN
 F 1 "GND" H 2983 2276 50  0000 C CNN
 F 2 "" H 2975 2450 50  0000 C CNN
@@
 $EndComp
 $Comp
-L GND #PWR49
+L GND #PWR062
 U 1 1 568BD87B
 P 3225 3050
-F 0 "#PWR49" H 3225 2800 50  0001 C CNN
+F 0 "#PWR062" H 3225 2800 50  0001 C CNN
 F 1 "GND" H 3233 2876 50  0000 C CNN
 F 2 "" H 3225 3050 50  0000 C CNN
@@
 F 0 "C12" H 4038 3996 50  0000 L CNN
 F 1 "100uF" H 4038 3904 50  0000 L CNN
-F 2 "armin-footprints:ELCO-8mm" H 3950 3950 50  0001 C CNN
+F 2 "capacitors:ELCO-8mm-3.5mm_pitch" H 3950 3950 50  0001 C CNN
 F 3 "" H 3950 3950 50  0000 C CNN
 	1    3950 3950
@@
 $EndComp
 $Comp
-L Vsupply #P16
+L Vsupply #P063
 U 1 1 568BDFCA
 P 3125 3300
-F 0 "#P16" H 3125 3300 60  0001 C CNN
+F 0 "#P063" H 3125 3300 60  0001 C CNN
 F 1 "Vsupply" H 3125 3250 34  0000 C CNN
 F 2 "" H 3125 3300 60  0000 C CNN
@@
 	1125 3650 1125 3950
 $Comp
-L +3.3V #PWR38
+L +3.3V #PWR064
 U 1 1 568BDFDB
 P 1125 3650
-F 0 "#PWR38" H 1125 3500 50  0001 C CNN
+F 0 "#PWR064" H 1125 3500 50  0001 C CNN
 F 1 "+3.3V" H 1143 3824 50  0000 C CNN
 F 2 "" H 1125 3650 50  0000 C CNN
@@
 $EndComp
 $Comp
-L +3.3V #PWR44
+L +3.3V #PWR065
 U 1 1 568BDFE7
 P 3025 4250
-F 0 "#PWR44" H 3025 4100 50  0001 C CNN
+F 0 "#PWR065" H 3025 4100 50  0001 C CNN
 F 1 "+3.3V" H 3025 4375 50  0000 C CNN
 F 2 "" H 3025 4250 50  0000 C CNN
@@
 	2875 4250 3025 4250
 $Comp
-L GND #PWR41
+L GND #PWR066
 U 1 1 568BDFEE
 P 2950 3750
-F 0 "#PWR41" H 2950 3500 50  0001 C CNN
+F 0 "#PWR066" H 2950 3500 50  0001 C CNN
 F 1 "GND" H 2958 3576 50  0000 C CNN
 F 2 "" H 2950 3750 50  0000 C CNN
@@
 $EndComp
 $Comp
-L GND #PWR47
+L GND #PWR067
 U 1 1 568BDFF4
 P 3200 4350
-F 0 "#PWR47" H 3200 4100 50  0001 C CNN
+F 0 "#PWR067" H 3200 4100 50  0001 C CNN
 F 1 "GND" H 3208 4176 50  0000 C CNN
 F 2 "" H 3200 4350 50  0000 C CNN
@@
 F 0 "C15" H 8988 4121 50  0000 L CNN
 F 1 "100uF" H 8988 4029 50  0000 L CNN
-F 2 "armin-footprints:ELCO-8mm" H 8900 4075 50  0001 C CNN
+F 2 "capacitors:ELCO-8mm-3.5mm_pitch" H 8900 4075 50  0001 C CNN
 F 3 "" H 8900 4075 50  0000 C CNN
 	1    8900 4075
@@
 $EndComp
 $Comp
-L Vsupply #P21
+L Vsupply #P068
 U 1 1 568C39F8
 P 8250 3425
-F 0 "#P21" H 8250 3425 60  0001 C CNN
+F 0 "#P068" H 8250 3425 60  0001 C CNN
 F 1 "Vsupply" H 8250 3375 34  0000 C CNN
 F 2 "" H 8250 3425 60  0000 C CNN
@@
 	6250 4075 6250 3775
 $Comp
-L +3.3V #PWR52
+L +3.3V #PWR069
 U 1 1 568C3A09
 P 6250 3775
-F 0 "#PWR52" H 6250 3625 50  0001 C CNN
+F 0 "#PWR069" H 6250 3625 50  0001 C CNN
 F 1 "+3.3V" H 6268 3949 50  0000 C CNN
 F 2 "" H 6250 3775 50  0000 C CNN
@@
 $EndComp
 $Comp
-L +3.3V #PWR58
+L +3.3V #PWR070
 U 1 1 568C3A15
 P 8150 4375
-F 0 "#PWR58" H 8150 4225 50  0001 C CNN
+F 0 "#PWR070" H 8150 4225 50  0001 C CNN
 F 1 "+3.3V" H 8150 4500 50  0000 C CNN
 F 2 "" H 8150 4375 50  0000 C CNN
@@
 	8000 4375 8150 4375
 $Comp
-L GND #PWR55
+L GND #PWR071
 U 1 1 568C3A1C
 P 8075 3875
-F 0 "#PWR55" H 8075 3625 50  0001 C CNN
+F 0 "#PWR071" H 8075 3625 50  0001 C CNN
 F 1 "GND" H 8083 3701 50  0000 C CNN
 F 2 "" H 8075 3875 50  0000 C CNN
@@
 $EndComp
 $Comp
-L GND #PWR61
+L GND #PWR072
 U 1 1 568C3A22
 P 8325 4475
-F 0 "#PWR61" H 8325 4225 50  0001 C CNN
+F 0 "#PWR072" H 8325 4225 50  0001 C CNN
 F 1 "GND" H 8333 4301 50  0000 C CNN
 F 2 "" H 8325 4475 50  0000 C CNN
@@
 F 0 "C16" H 8963 1446 50  0000 L CNN
 F 1 "100uF" H 8963 1354 50  0000 L CNN
-F 2 "armin-footprints:ELCO-8mm" H 8875 1400 50  0001 C CNN
+F 2 "capacitors:ELCO-8mm-3.5mm_pitch" H 8875 1400 50  0001 C CNN
 F 3 "" H 8875 1400 50  0000 C CNN
 	1    8875 1400
@@
 $EndComp
 $Comp
-L Vsupply #P19
+L Vsupply #P073
 U 1 1 568C3E5C
 P 8225 750
-F 0 "#P19" H 8225 750 60  0001 C CNN
+F 0 "#P073" H 8225 750 60  0001 C CNN
 F 1 "Vsupply" H 8225 700 34  0000 C CNN
 F 2 "" H 8225 750 60  0000 C CNN
@@
 	6225 1100 6225 1400
 $Comp
-L +3.3V #PWR50
+L +3.3V #PWR074
 U 1 1 568C3E6D
 P 6225 1100
-F 0 "#PWR50" H 6225 950 50  0001 C CNN
+F 0 "#PWR074" H 6225 950 50  0001 C CNN
 F 1 "+3.3V" H 6243 1274 50  0000 C CNN
 F 2 "" H 6225 1100 50  0000 C CNN
@@
 $EndComp
 $Comp
-L +3.3V #PWR56
+L +3.3V #PWR075
 U 1 1 568C3E79
 P 8125 1700
-F 0 "#PWR56" H 8125 1550 50  0001 C CNN
+F 0 "#PWR075" H 8125 1550 50  0001 C CNN
 F 1 "+3.3V" H 8125 1825 50  0000 C CNN
 F 2 "" H 8125 1700 50  0000 C CNN
@@
 	7975 1700 8125 1700
 $Comp
-L GND #PWR53
+L GND #PWR076
 U 1 1 568C3E80
 P 8050 1200
-F 0 "#PWR53" H 8050 950 50  0001 C CNN
+F 0 "#PWR076" H 8050 950 50  0001 C CNN
 F 1 "GND" H 8058 1026 50  0000 C CNN
 F 2 "" H 8050 1200 50  0000 C CNN
@@
 $EndComp
 $Comp
-L GND #PWR59
+L GND #PWR077
 U 1 1 568C3E86
 P 8300 1800
-F 0 "#PWR59" H 8300 1550 50  0001 C CNN
+F 0 "#PWR077" H 8300 1550 50  0001 C CNN
 F 1 "GND" H 8308 1626 50  0000 C CNN
 F 2 "" H 8300 1800 50  0000 C CNN
@@
 F 0 "C17" H 8963 2821 50  0000 L CNN
 F 1 "100uF" H 8963 2729 50  0000 L CNN
-F 2 "armin-footprints:ELCO-8mm" H 8875 2775 50  0001 C CNN
+F 2 "capacitors:ELCO-8mm-3.5mm_pitch" H 8875 2775 50  0001 C CNN
 F 3 "" H 8875 2775 50  0000 C CNN
 	1    8875 2775
@@
 $EndComp
 $Comp
-L Vsupply #P20
+L Vsupply #P078
 U 1 1 568C4325
 P 8225 2125
-F 0 "#P20" H 8225 2125 60  0001 C CNN
+F 0 "#P078" H 8225 2125 60  0001 C CNN
 F 1 "Vsupply" H 8225 2075 34  0000 C CNN
 F 2 "" H 8225 2125 60  0000 C CNN
@@
 	6225 2475 6225 2775
 $Comp
-L +3.3V #PWR51
+L +3.3V #PWR079
 U 1 1 568C4336
 P 6225 2475
-F 0 "#PWR51" H 6225 2325 50  0001 C CNN
+F 0 "#PWR079" H 6225 2325 50  0001 C CNN
 F 1 "+3.3V" H 6243 2649 50  0000 C CNN
 F 2 "" H 6225 2475 50  0000 C CNN
@@
 $EndComp
 $Comp
-L +3.3V #PWR57
+L +3.3V #PWR080
 U 1 1 568C4342
 P 8125 3075
-F 0 "#PWR57" H 8125 2925 50  0001 C CNN
+F 0 "#PWR080" H 8125 2925 50  0001 C CNN
 F 1 "+3.3V" H 8125 3200 50  0000 C CNN
 F 2 "" H 8125 3075 50  0000 C CNN
@@
 	7975 3075 8125 3075
 $Comp
-L GND #PWR54
+L GND #PWR081
 U 1 1 568C4349
 P 8050 2575
-F 0 "#PWR54" H 8050 2325 50  0001 C CNN
+F 0 "#PWR081" H 8050 2325 50  0001 C CNN
 F 1 "GND" H 8058 2401 50  0000 C CNN
 F 2 "" H 8050 2575 50  0000 C CNN
@@
 $EndComp
 $Comp
-L GND #PWR60
+L GND #PWR082
 U 1 1 568C434F
 P 8300 3175
-F 0 "#PWR60" H 8300 2925 50  0001 C CNN
+F 0 "#PWR082" H 8300 2925 50  0001 C CNN
 F 1 "GND" H 8308 3001 50  0000 C CNN
 F 2 "" H 8300 3175 50  0000 C CNN
