File: steppers.sch (KiCad schematic (older format))
At the start: 24 parts, among them J1 HEADER, J10 STEPSTICK, J11 STEPSTICK, J12 STEPSTICK, J2 HEADER, J3 HEADER, J4 STEPSTICK, J5 STEPSTICK, J6 STEPSTICK, J7 HEADER, J8 HEADER, J9 HEADER, P10 CONN_01X04, P11 CONN_01X04, P12 CONN_01X04, P7 CONN_02X04, P8 CONN_01X04, P9 CONN_01X04

Commit message: fixed minor issue
Parts:
- J1, J2, J3, J7, J8, J9: footprint armin-footprints:CON_HDR_2x3_2.54mm -> headers:CON_HDR_2x3_2.54mm
- P10, P11, P12, P8, P9: footprint armin-footprints:CON_HDR_1x4_2.54mm -> headers:CON_HDR_1x4_2.54mm
- P7: footprint armin-footprints:CON_HDR_2x4_2.54mm -> headers:CON_HDR_2x4_2.54mm
Changed lines of the file:
@@
 F 0 "J2" H 1675 1907 34  0000 C CNN
 F 1 "HEADER" H 1675 1838 34  0000 C CNN
-F 2 "armin-footprints:CON_HDR_2x3_2.54mm" H 1500 1475 60  0001 C CNN
+F 2 "headers:CON_HDR_2x3_2.54mm" H 1500 1475 60  0001 C CNN
 F 3 "" H 1500 1475 60  0000 C CNN
 	1    1500 1475
@@
 F 0 "P8" H 3477 1513 50  0000 L CNN
 F 1 "CONN_01X04" H 3477 1421 50  0000 L CNN
-F 2 "armin-footprints:CON_HDR_1x4_2.54mm" H 3400 1475 50  0001 C CNN
+F 2 "headers:CON_HDR_1x4_2.54mm" H 3400 1475 50  0001 C CNN
 F 3 "" H 3400 1475 50  0000 C CNN
 	1    3400 1475
@@
 F 0 "J3" H 1675 3132 34  0000 C CNN
 F 1 "HEADER" H 1675 3063 34  0000 C CNN
-F 2 "armin-footprints:CON_HDR_2x3_2.54mm" H 1500 2700 60  0001 C CNN
+F 2 "headers:CON_HDR_2x3_2.54mm" H 1500 2700 60  0001 C CNN
 F 3 "" H 1500 2700 60  0000 C CNN
 	1    1500 2700
@@
 F 0 "P9" H 3477 2738 50  0000 L CNN
 F 1 "CONN_01X04" H 3477 2646 50  0000 L CNN
-F 2 "armin-footprints:CON_HDR_1x4_2.54mm" H 3400 2700 50  0001 C CNN
+F 2 "headers:CON_HDR_1x4_2.54mm" H 3400 2700 50  0001 C CNN
 F 3 "" H 3400 2700 50  0000 C CNN
 	1    3400 2700
@@
 F 0 "J7" H 6775 4557 34  0000 C CNN
 F 1 "HEADER" H 6775 4488 34  0000 C CNN
-F 2 "armin-footprints:CON_HDR_2x3_2.54mm" H 6600 4125 60  0001 C CNN
+F 2 "headers:CON_HDR_2x3_2.54mm" H 6600 4125 60  0001 C CNN
 F 3 "" H 6600 4125 60  0000 C CNN
 	1    6600 4125
@@
 F 0 "P10" H 8577 4163 50  0000 L CNN
 F 1 "CONN_01X04" H 8577 4071 50  0000 L CNN
-F 2 "armin-footprints:CON_HDR_1x4_2.54mm" H 8500 4125 50  0001 C CNN
+F 2 "headers:CON_HDR_1x4_2.54mm" H 8500 4125 50  0001 C CNN
 F 3 "" H 8500 4125 50  0000 C CNN
 	1    8500 4125
@@
 F 0 "J8" H 6750 1882 34  0000 C CNN
 F 1 "HEADER" H 6750 1813 34  0000 C CNN
-F 2 "armin-footprints:CON_HDR_2x3_2.54mm" H 6575 1450 60  0001 C CNN
+F 2 "headers:CON_HDR_2x3_2.54mm" H 6575 1450 60  0001 C CNN
 F 3 "" H 6575 1450 60  0000 C CNN
 	1    6575 1450
@@
 F 0 "P11" H 8552 1488 50  0000 L CNN
 F 1 "CONN_01X04" H 8552 1396 50  0000 L CNN
-F 2 "armin-footprints:CON_HDR_1x4_2.54mm" H 8475 1450 50  0001 C CNN
+F 2 "headers:CON_HDR_1x4_2.54mm" H 8475 1450 50  0001 C CNN
 F 3 "" H 8475 1450 50  0000 C CNN
 	1    8475 1450
@@
 F 0 "J9" H 6750 3257 34  0000 C CNN
 F 1 "HEADER" H 6750 3188 34  0000 C CNN
-F 2 "armin-footprints:CON_HDR_2x3_2.54mm" H 6575 2825 60  0001 C CNN
+F 2 "headers:CON_HDR_2x3_2.54mm" H 6575 2825 60  0001 C CNN
 F 3 "" H 6575 2825 60  0000 C CNN
 	1    6575 2825
@@
 F 0 "P12" H 8552 2863 50  0000 L CNN
 F 1 "CONN_01X04" H 8552 2771 50  0000 L CNN
-F 2 "armin-footprints:CON_HDR_1x4_2.54mm" H 8475 2825 50  0001 C CNN
+F 2 "headers:CON_HDR_1x4_2.54mm" H 8475 2825 50  0001 C CNN
 F 3 "" H 8475 2825 50  0000 C CNN
 	1    8475 2825
@@
 F 0 "P7" H 3425 4250 50  0000 C CNN
 F 1 "CONN_02X04" H 3425 3750 50  0000 C CNN
-F 2 "armin-footprints:CON_HDR_2x4_2.54mm" H 3425 2800 50  0001 C CNN
+F 2 "headers:CON_HDR_2x4_2.54mm" H 3425 2800 50  0001 C CNN
 F 3 "" H 3425 2800 50  0000 C CNN
 	1    3425 4000
@@
 F 0 "J1" H 1650 4432 34  0000 C CNN
 F 1 "HEADER" H 1650 4363 34  0000 C CNN
-F 2 "armin-footprints:CON_HDR_2x3_2.54mm" H 1475 4000 60  0001 C CNN
+F 2 "headers:CON_HDR_2x3_2.54mm" H 1475 4000 60  0001 C CNN
 F 3 "" H 1475 4000 60  0000 C CNN
 	1    1475 4000

Commit message: fixed some errors
Parts:
- J10, J11, J12, J4, J5, J6: footprint armin-footprints:STEPSTICK -> misc:STEPSTICK
Changed lines of the file:
@@
 F 0 "J5" H 2475 2750 34  0000 C CNN
 F 1 "STEPSTICK" H 2475 2650 34  0000 C CNN
-F 2 "armin-footprints:STEPSTICK" H 2025 1925 60  0001 C CNN
+F 2 "misc:STEPSTICK" H 2025 1925 60  0001 C CNN
 F 3 "" H 2025 1925 60  0000 C CNN
 	1    2025 1925
@@
 F 0 "J6" H 2475 3975 34  0000 C CNN
 F 1 "STEPSTICK" H 2475 3875 34  0000 C CNN
-F 2 "armin-footprints:STEPSTICK" H 2025 3150 60  0001 C CNN
+F 2 "misc:STEPSTICK" H 2025 3150 60  0001 C CNN
 F 3 "" H 2025 3150 60  0000 C CNN
 	1    2025 3150
@@
 F 0 "J4" H 2450 5275 34  0000 C CNN
 F 1 "STEPSTICK" H 2450 5175 34  0000 C CNN
-F 2 "armin-footprints:STEPSTICK" H 2000 4450 60  0001 C CNN
+F 2 "misc:STEPSTICK" H 2000 4450 60  0001 C CNN
 F 3 "" H 2000 4450 60  0000 C CNN
 	1    2000 4450
@@
 F 0 "J10" H 7575 5400 34  0000 C CNN
 F 1 "STEPSTICK" H 7575 5300 34  0000 C CNN
-F 2 "armin-footprints:STEPSTICK" H 7125 4575 60  0001 C CNN
+F 2 "misc:STEPSTICK" H 7125 4575 60  0001 C CNN
 F 3 "" H 7125 4575 60  0000 C CNN
 	1    7125 4575
@@
 F 0 "J11" H 7550 2725 34  0000 C CNN
 F 1 "STEPSTICK" H 7550 2625 34  0000 C CNN
-F 2 "armin-footprints:STEPSTICK" H 7100 1900 60  0001 C CNN
+F 2 "misc:STEPSTICK" H 7100 1900 60  0001 C CNN
 F 3 "" H 7100 1900 60  0000 C CNN
 	1    7100 1900
@@
 F 0 "J12" H 7550 4100 34  0000 C CNN
 F 1 "STEPSTICK" H 7550 4000 34  0000 C CNN
-F 2 "armin-footprints:STEPSTICK" H 7100 3275 60  0001 C CNN
+F 2 "misc:STEPSTICK" H 7100 3275 60  0001 C CNN
 F 3 "" H 7100 3275 60  0000 C CNN
 	1    7100 3275
